File: pcb/kicad/keyboard_kicad.kicad_pcb (KiCad board)
At the start: 2 copper layers, 349.7 x 122 mm, 173 parts, among them SW1 SW_Push, SW10 SW_Push, SW11 SW_Push, SW12 SW_Push, SW13 SW_Push, SW14 SW_Push, SW15 SW_Push, SW16 SW_Push, SW17 SW_Push, SW18 SW_Push, SW19 SW_Push, SW2 SW_Push, SW20 SW_Push, SW21 SW_Push, SW22 SW_Push, SW23 SW_Push, SW24 SW_Push, SW25 SW_Push, SW26 SW_Push, SW27 SW_Push, SW28 SW_Push, SW29 SW_Push, SW3 SW_Push, SW30 SW_Push, SW31 SW_Push, SW32 SW_Push, SW33 SW_Push, SW34 SW_Push, SW35 SW_Push, SW36 SW_Push, SW37 SW_Push, SW38 SW_Push, SW39 SW_Push, SW4 SW_Push, SW40 SW_Push, SW41 SW_Push, SW42 SW_Push, SW43 SW_Push, SW44 SW_Push, SW45 SW_Push, SW46 SW_Push, SW47 SW_Push, SW48 SW_Push, SW49 SW_Push, SW5 SW_Push, SW50 SW_Push, SW51 SW_Push, SW52 SW_Push, SW53 SW_Push, SW54 SW_Push, SW55 SW_Push, SW56 SW_Push, SW57 SW_Push, SW58 SW_Push, SW59 SW_Push, SW6 SW_Push, SW60 SW_Push, SW61 SW_Push, SW62 SW_Push, SW63 SW_Push, SW64 SW_Push, SW65 SW_Push, SW66 SW_Push, SW67 SW_Push, SW68 SW_Push, SW69 SW_Push, SW7 SW_Push, SW70 SW_Push, SW71 SW_Push, SW72 SW_Push, SW73 SW_Push, SW74 SW_Push, SW75 SW_Push, SW76 SW_Push, SW77 SW_Push, SW78 SW_Push, SW79 SW_Push, SW8 SW_Push, SW80 SW_Push, SW81 SW_Push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

Commit message: Add files via upload
Parts:
- removed H1, H2 (x2), H3, H4 (x2): MountingHole, MountingHole:MountingHole_2mm
- SW78: footprint ScottoKeebs_Stabilizer:Stabilizer_MX_6.25u -> Stabilizers:Stabilizer_Cherry_MX_6.25u
- U1: moved to B.Cu
- moved D69 2.38 mm to (383.9, 173.2)
- moved SW45 2.38 mm to (374.4, 170.1)
- moved SW61 0.58 mm to (124.4, 207.7)
- moved SW59 0.58 mm to (367.3, 188.6)
- moved SW78 0.51 mm to (257.7, 227.3)
- moved SW72 0.07 mm to (362.4, 208.3)
- turned U1 to 180 degrees
Routing:
- net Column 15: track 213.4 -> 116.6 mm, vias 2 -> 0
- net Column 12: track 278.9 -> 184.0 mm, vias 2 -> 4
- net Column 13: track 257.8 -> 165.2 mm, vias 2 -> 4
- net Column 11: track 293.3 -> 206.8 mm, vias 2 -> 4
- net Column 14: track 246.2 -> 167.0 mm
- net Column 10: track 279.2 -> 225.1 mm
- net Column 6: track 364.9 -> 315.1 mm, vias 2 -> 4
- net Column 0: track 503.0 -> 461.8 mm
- net Column 5: track 384.0 -> 346.9 mm, vias 4 -> 5
- net Column 2: track 453.2 -> 421.8 mm
- net Column 3: track 432.8 -> 403.7 mm
- net Column 1: track 463.7 -> 437.3 mm
- net Row 0: track 313.0 -> 330.5 mm, vias 30 -> 0
- net Column 4: track 547.9 -> 563.2 mm, vias 2 -> 4
- net Row 2: track 333.9 -> 344.4 mm, vias 28 -> 0
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Other:
- board size 349.7 x 122 mm -> 349.1 x 122 mm
