File: pcb/kicad/keyboard_kicad.kicad_sch (KiCad schematic)
At the start: 171 parts, among them SW1 SW_Push, SW10 SW_Push, SW11 SW_Push, SW12 SW_Push, SW13 SW_Push, SW14 SW_Push, SW15 SW_Push, SW16 SW_Push, SW17 SW_Push, SW18 SW_Push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

Commit message: Add files via upload
Parts:
- removed H1, H2, H3, H4: MountingHole, MountingHole:MountingHole_2mm, symbol Mechanical:MountingHole
- SW78: footprint ScottoKeebs_Stabilizer:Stabilizer_MX_6.25u -> Stabilizers:Stabilizer_Cherry_MX_6.25u
